Commit message: test

File: src/ezmower_robot/urdf/robot_core.urdf (robot description, URDF)
Before this commit: robot None, 9 links, 10 joints
Links:
- link chasis: geometry collision box size=${chasis_height} ${chasis_width} ${chasis_depth}; visual mesh filename=file://$(find ezmower_robot)/meshes/chasis.stl scale=0.0001 0.0001 0.0001

Commit message: rotated lidar-link

File: src/ezmower_robot/urdf/robot_core.urdf (robot description, URDF)
Before this commit: robot None, 9 links, 10 joints
Joints:
- joint lidar_joint: origin xyz=0 0 0.012 -> xyz=0 0 0.012 rpy=0.0 0.0 ${pi}

Commit message: nav2 navigateToGoal working

File: src/ezmower_robot/urdf/robot_core.urdf (robot description, URDF)
Before this commit: robot None, 9 links, 10 joints
Links:
- link chasis: geometry collision box size=${chasis_height} ${chasis_width} ${chasis_depth}; visual mesh filename=package://ezmower_robot/meshes/chasis.stl scale=0.0001 0.0001 0.0001

Commit message: fixed some rviz configs

File: src/ezmower_robot/urdf/robot_core.urdf (robot description, URDF)
Before this commit: robot None, 9 links, 10 joints
Links:
- link roof_link: geometry collision box size=${chasis_height} ${chasis_width} 0.005; visual mesh filename=package://ezmower_robot/meshes/top_cover.stl scale=0.001 0.001 0.001
